Commit message: some changes to teh models and launch files

File: src/robot_description/urdf/robot.urdf (robot description, URDF)
Before this commit: robot my_robot, 6 links, 5 joints
Links:
- removed link depth_camera_link
- added link camera_link, mass .01; collision box size=.025 .09 .025; visual box size=.09 .025 .025
Joints:
- joint dc_joint: child depth_camera_link -> camera_link
